File: kicad/pynqsdr/pynqsdr.kicad_pcb (KiCad board)
At the start: 4 copper layers, 96.9 x 71.6 mm, 180 parts, among them J1 Header 6X2, J2J3 Header 8X2, J4 Header 8X2, J7 Header 8, T1 TCM1-63AX+, T2 TCM1-63AX+, T3 TCM1-63AX+, T4 TCM1-63AX+, U11 TPS7A8101, U12 TPS7A8101, U5 AD9363, X1 40MHz, X4 40MHz

Commit message: v1.1 update
Parts:
- removed 1VXG1: Header 2, PYNQSDR:HDR1X2
- removed C41, C42, C43, C44, C45, C46, C49, C50, C51, C52, C53, C54, C55, C56, C57, C61: 0.1μ, PYNQSDR:LC-0402_C
- removed C64: 10μ, PYNQSDR:LC-0402_C
- removed CP2, CP5: 22pF, PYNQSDR:LC-0402_C
- removed CP4, CP6: 22uF, PYNQSDR:LC-0805_C
- removed Ct1, Ct2: 3.3nF, PYNQSDR:PCBComponent_1
- removed LP2: 4.7uH, PYNQSDR:L1008
- removed R28, R30, R31, R33, R34, R36, R37, R39, R40, R42, R43, R45, R46, R48, R49, R51, R52, R54, R55, R57, R58, R60, R61, R63, R64, R66, R67, R69, R70, R72, R76, R78, RP3: 10K, PYNQSDR:LC-0402_R
- removed RP4: 20K, PYNQSDR:LC-0402_R
- removed RP5, RP6: NC, PYNQSDR:LC-0402_R
- removed RX22: 0R, PYNQSDR:LC-0402_R
- removed TX3: JCCEM001, PYNQSDR:CNSMARAL687W375H171
- removed TX_SMT1: U.FL-R-SMT_10_, PYNQSDR:UFLRSMT10
- removed UP2: AP3419, PYNQSDR:AP3419
- added C10: 0.1μ, PYNQSDR:LC-0402_C, B.Cu at (111.2, 94.2)
- added C11: 0.1μ, PYNQSDR:LC-0402_C, B.Cu at (123.0, 90.1)
- added C4: 0.1μ, PYNQSDR:LC-0402_C, B.Cu at (115.8, 89.1)
- added C5: 0.1μ, PYNQSDR:LC-0402_C, B.Cu at (106.7, 89.6)
- added C6: 0.1μ, PYNQSDR:LC-0402_C, B.Cu at (119.3, 89.1)
- added C7: 0.1μ, PYNQSDR:LC-0402_C, B.Cu at (102.8, 89.6)
- added C8: 0.1μ, PYNQSDR:LC-0402_C, B.Cu at (109.1, 82.9)
- added C9: 0.1μ, PYNQSDR:LC-0402_C, B.Cu at (125.6, 90.1)
- added R10: 100R, PYNQSDR:LC-0402_R, F.Cu at (115.8, 94.3)
- added R11: 100R, PYNQSDR:LC-0402_R, F.Cu at (127.3, 94.3)
- added R12: 100R, PYNQSDR:LC-0402_R, F.Cu at (111.4, 100.1)
- added R13: 100R, PYNQSDR:LC-0402_R, F.Cu at (107.8, 100.1)
- added R14: 100R, PYNQSDR:LC-0402_R, F.Cu at (103.8, 100.1)
- added R15: 100R, PYNQSDR:LC-0402_R, B.Cu at (111.6, 88.3)
- added R16: 0R, PYNQSDR:LC-0402_R, F.Cu at (184.5, 107.9)
- added R8: 100R, PYNQSDR:LC-0402_R, F.Cu at (123.5, 94.3)
- added R9: 100R, PYNQSDR:LC-0402_R, F.Cu at (119.6, 94.3)
- added U10: sn65cml100, Package_SO:TSSOP-8_4.4x3mm_P0.65mm, F.Cu at (103.8, 94.9)
- added U13: sn65cml100, Package_SO:TSSOP-8_4.4x3mm_P0.65mm, F.Cu at (111.6, 86.7)
- added U3: sn65cml100, Package_SO:TSSOP-8_4.4x3mm_P0.65mm, F.Cu at (123.4, 88.7)
- added U4: sn65cml100, Package_SO:TSSOP-8_4.4x3mm_P0.65mm, F.Cu at (119.6, 88.7)
- added U6: sn65cml100, Package_SO:TSSOP-8_4.4x3mm_P0.65mm, F.Cu at (115.8, 88.7)
- added U7: sn65cml100, Package_SO:TSSOP-8_4.4x3mm_P0.65mm, F.Cu at (127.3, 88.7)
- added U8: sn65cml100, Package_SO:TSSOP-8_4.4x3mm_P0.65mm, F.Cu at (111.6, 94.8)
- added U9: sn65cml100, Package_SO:TSSOP-8_4.4x3mm_P0.65mm, F.Cu at (107.8, 94.9)
- C143: value 0.1μ -> 0.1μ NC
- C144: value 10μ -> 10μ NC
- C33: value 1nF -> 1nF NC
- C62: value 10μ -> NC
- J2J3: value Header 8X2 -> Header 4X2
- R2: value 1MΩ -> 1MΩ NC
- RX4: value 0R -> NC
- X1: value 40MHz -> 30MHz
- X4: value 40MHz -> 40MHz NC
- moved X4 1.52 mm to (146.0, 100.2)
- moved X1 1.47 mm to (180.9, 108.3)
- moved RX3 0.25 mm to (102.8, 132.5)
- moved RX_SMT1 0.25 mm to (109.7, 132.5)
Connections:
- net Net-(C152-Pad2) renamed /XTAL1V8_IN
- HDMI1 pad 1: /RX_D2_P -> /TMDS_D3_P
- HDMI1 pad 10: /RX_D5_P -> /TMDS_CLK_P
- HDMI1 pad 12: /RX_D5_N -> /TMDS_CLK_N
- HDMI1 pad 3: /RX_D2_N -> /TMDS_D3_N
- HDMI1 pad 4: /RX_D4_P -> /TMDS_D1_P
- HDMI1 pad 6: /RX_D4_N -> /TMDS_D1_N
- HDMI1 pad 7: /RX_D0_P -> /TMDS_FRAME_P
- HDMI1 pad 9: /RX_D0_N -> /TMDS_FRAME_N
- HDMI2 pad 1: /RX_FRAME_P -> /TMDS_D5_P
- HDMI2 pad 10: /RX_D3_P -> /TMDS_D2_P
- HDMI2 pad 12: /RX_D3_N -> /TMDS_D2_N
- HDMI2 pad 3: /RX_FRAME_N -> /TMDS_D5_N
- HDMI2 pad 4: /RX_D1_P -> /TMDS_D0_P
- HDMI2 pad 6: /RX_D1_N -> /TMDS_D0_N
- HDMI2 pad 7: /DATA_CLK_P -> /TMDS_D4_P
- HDMI2 pad 9: /DATA_CLK_N -> /TMDS_D4_N
- PMODB1 pad 5: /Q3_P -> /FB_CLK_P
- PMODB1 pad 7: /Q3_N -> /FB_CLK_N
- U5 pad D10: /TX_D4_N -> /P3_P
- U5 pad D11: /TX_D5_N -> /P4_P
- U5 pad D7: /TX_D1_N -> /Q4_P
- U5 pad D8: /TX_D2_N -> /P1_P
- U5 pad D9: /TX_D3_N -> /Q2_P
- U5 pad E10: /TX_D3_P -> /Q2_N
- U5 pad E11: /TX_D4_P -> /P3_N
- U5 pad E12: /TX_D5_P -> /P4_N
- U5 pad E7: /TX_D0_N -> /P2_P
- U5 pad E8: /TX_D1_P -> /Q4_N
- U5 pad E9: /TX_D2_P -> /P1_N
- U5 pad F8: /TX_D0_P -> /P2_N
- U5 pad G9: /TX_FRAME_P -> /Q1_P
- U5 pad H9: /TX_FRAME_N -> /Q1_N
Routing:
- net VCC1P5: track 114.1 -> 0.00 mm, vias 15 -> 0
- net /Q4_P: track 8.51 -> 68.6 mm, vias 0 -> 2
- net /Q4_N: track 8.46 -> 67.3 mm, vias 0 -> 2
- net /TX_D1_N: track 55.2 -> 0.00 mm, vias 2 -> 0
- net /TX_FRAME_P: track 54.9 -> 0.00 mm, vias 2 -> 0
- net /TX_FRAME_N: track 54.1 -> 0.00 mm, vias 2 -> 0
- net /TX_D1_P: track 53.7 -> 0.00 mm, vias 2 -> 0
- net /Q2_P: track 7.65 -> 58.3 mm, vias 0 -> 3
- net /Q2_N: track 8.05 -> 58.3 mm, vias 0 -> 3
- net /Q1_P: track 8.68 -> 56.3 mm, vias 0 -> 2
- net /TX_D3_P: track 47.2 -> 0.00 mm, vias 2 -> 0
- net /TX_D3_N: track 47.1 -> 0.00 mm, vias 2 -> 0
- net /Q1_N: track 9.06 -> 55.9 mm, vias 0 -> 2
- net /XTAL1V8_IN: track 2.28 -> 45.1 mm, vias 0 -> 4
- net /TX_D2_N: track 42.6 -> 0.00 mm, vias 3 -> 0
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- removed copper zone on F.Cu, net RFGND1
- removed copper zone on In1.Cu, net RFGND1
Other:
- board text added: "1V8 G"
- board text added: "3V3 G"
- board text added: "5V0 G"
- board text added: "RX"
- board text added: "TX"
- board text added: "v1.1 happy lunar new year 2022.1"
- board text removed: "2021.10 Trick or treat"

Commit message: V1.2 update
Parts:
- removed C11, C9: 0.1μ, PYNQSDR:LC-0402_C
- added C2: 0.1μ, PYNQSDR:LC-0402_C, F.Cu at (175.9, 122.5)
- added C3: NC, PYNQSDR:LC-0402_C, F.Cu at (178.9, 125.7)
- added R1: NC, PYNQSDR:LC-0402_R, B.Cu at (178.7, 106.8)
- added X2: TCXO, Crystal:Crystal_SMD_7050-4Pin_7.0x5.0mm, F.Cu at (179.8, 120.1)
- C33, R2: moved to B.Cu
- HDMI1, HDMI2: value ${ALTIUM_VALUE} -> HDMI_A
- RX1, RX3, TX1: value JCCEM001 -> Conn_Coaxial; footprint PYNQSDR:CNSMARAL687W375H171 -> Connector_Coaxial:SMA_Amphenol_132289_EdgeMount
- U10, U13, U3, U4, U6, U7, U8, U9: footprint Package_SO:TSSOP-8_4.4x3mm_P0.65mm -> Package_SO:TSSOP-8_3x3mm_P0.65mm
- moved R15 1.73 mm to (111.6, 90.0)
- moved R9 0.76 mm to (119.6, 93.5)
- moved R10 0.76 mm to (115.8, 93.6)
- moved R8 0.76 mm to (123.4, 93.5)
- moved R11 0.76 mm to (127.3, 93.5)
- moved C10 0.73 mm to (111.2, 94.9)
- moved C5 0.69 mm to (106.7, 90.3)
- moved C7 0.55 mm to (102.8, 90.1)
- moved R13 0.39 mm to (107.8, 99.7)
- moved R14 0.33 mm to (103.8, 99.8)
- moved R12 0.28 mm to (111.4, 99.8)
- moved R2 0.15 mm to (120.3, 75.4)
- moved C8 0.10 mm to (109.1, 83.0)
- moved RX_SMT2 0.08 mm to (186.8, 102.8)
- moved TX_SMT2 0.07 mm to (186.9, 125.4)
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Routing:
- net GND: track 120.5 -> 174.6 mm, vias 75 -> 84
- net Net-(R1-Pad2): track 0.00 -> 12.9 mm, vias 0 -> 1
- net /RX_D3_N: track 49.7 -> 47.1 mm
- net VCC_3V3: track 50.6 -> 53.0 mm
- net /RX_D3_P: track 49.0 -> 46.7 mm
- net /RX_D2_N: track 50.2 -> 48.6 mm
- net /RX_D2_P: track 49.4 -> 48.0 mm
- net /OI2: track 21.8 -> 23.0 mm, vias 0 -> 1
- net /DATA_CLK_P: track 36.6 -> 35.8 mm
- net /RX_D1_P: track 31.4 -> 30.6 mm
- net /RX_D1_N: track 32.5 -> 31.8 mm
- net /DATA_CLK_N: track 37.0 -> 36.2 mm
- net /TMDS_D4_P: track 14.8 -> 15.5 mm
- net /TMDS_D4_N: track 14.7 -> 15.5 mm
- net /TMDS_FRAME_P: track 7.54 -> 8.25 mm
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Other:
- board text added: "KiCad version v1.0, converted from Altium so expect some tiny problems. I've run DRC and there's no real error. 2021.12.3, regymm So far no noticable problem from convertion, I'll purge any left Altium stuff found. 2022.9"
- board text added: "Some C/Rs unused, and will appear again when updating from sch Deleted unused on 2022.9"
- board text added: "v1.2 to the moon 2022.9"
- board text removed: "KiCad version v1.0, converted from Altium so expect some tiny problems. I've run DRC and there's no real error. 2021.12.3, regymm"
- board text removed: "Some C/Rs unused, and will appear again when updating from sch"
- board text removed: "v1.1 happy lunar new year 2022.1"
