File: kicad/pynqsdr/pynqsdr.kicad_sch (KiCad schematic)
At the start: 190 parts, among them J1 Header 6X2, J2J3 Header 8X2, J4 Header 8X2, J7 Header 8, T1 TCM1-63AX+, T2 TCM1-63AX+, T3 TCM1-63AX+, T4 TCM1-63AX+, U11 TPS7A8101, U12 TPS7A8101, U5 AD9363, X1 40MHz, X4 40MHz

Commit message: v1.1 update
Parts:
- removed 1VXG1: Header 2, PYNQSDR:HDR1X2, symbol pynqsdr-altium-import:0_Header 2
- removed C41, C42, C43, C44, C45, C46, C49, C50, C51, C52, C53, C54, C55, C56, C57, C61: 0.1μ, PYNQSDR:LC-0402_C, symbol pynqsdr-altium-import:2_CAP_2
- removed C64: 10μ, PYNQSDR:LC-0402_C, symbol pynqsdr-altium-import:0_CAP_2
- removed CP2, CP5: 22pF, PYNQSDR:LC-0402_C, symbol pynqsdr-altium-import:1_CAP_2
- removed CP4: 22uF, PYNQSDR:LC-0805_C, symbol pynqsdr-altium-import:0_CAP_1
- removed CP6: 22uF, PYNQSDR:LC-0805_C, symbol pynqsdr-altium-import:1_CAP_1
- removed Ct1, Ct2: 3.3nF, PYNQSDR:PCBComponent_1, symbol pynqsdr-altium-import:3_CAP_3_3
- removed LP2: 4.7uH, PYNQSDR:L1008, symbol pynqsdr-altium-import:0_INDUCTANCE
- removed R28, R30, R31, R33, R34, R36, R37, R39, R40, R42, R43, R45, R46, R48, R49, R51, R52, R54, R55, R57, R58, R60, R61, R63, R64, R66, R67, R69, R70, R72, R76, R78: 10K, PYNQSDR:LC-0402_R, symbol pynqsdr-altium-import:2_RES_1
- removed RP3: 10K, PYNQSDR:LC-0402_R, symbol pynqsdr-altium-import:1_RES_1
- removed RP4: 20K, PYNQSDR:LC-0402_R, symbol pynqsdr-altium-import:1_RES_1
- removed RP5, RP6: NC, PYNQSDR:LC-0402_R, symbol pynqsdr-altium-import:1_RES_1
- removed RX10, RX22: 0R, PYNQSDR:LC-0402_R, symbol pynqsdr-altium-import:2_RES_1
- removed TX3: JCCEM001, PYNQSDR:CNSMARAL687W375H171, symbol pynqsdr-altium-import:0_JCCEM001
- removed TX_SMT1: U.FL-R-SMT_10_, PYNQSDR:UFLRSMT10, symbol pynqsdr-altium-import:0_U.FL-R-SMT_10_
- removed UP2: AP3419, PYNQSDR:AP3419, symbol pynqsdr-altium-import:0_AP3419
- added C10, C11, C4, C5, C6, C7, C8, C9: 0.1μ, PYNQSDR:LC-0402_C, symbol pynqsdr-altium-import:1_CAP_2
- added R10, R11, R12, R13, R14, R15, R8, R9: 100R, PYNQSDR:LC-0402_R, symbol pynqsdr-altium-import:0_RES_1
- added R16: 0R, PYNQSDR:LC-0402_R, symbol pynqsdr-altium-import:2_RES_1
- added U10, U13, U3, U4, U6, U7, U8, U9: sn65cml100, Package_SO:TSSOP-8_4.4x3mm_P0.65mm, symbol New_Library:sn65cml100
- C143: value 0.1μ -> 0.1μ NC
- C144: value 10μ -> 10μ NC
- C33: value 1nF -> 1nF NC
- C62: value 10μ -> NC
- J2J3: value Header 8X2 -> Header 4X2
- R2: value 1MΩ -> 1MΩ NC
- RX4: value 0R -> NC
- X1: value 40MHz -> 30MHz
- X4: value 40MHz -> 40MHz NC
Connections:
- net Q3_N is gone; now on net FB_CLK_N: PMODB1.7
- net Q3_P is gone; now on net FB_CLK_P: PMODB1.5
- net TX_D0_N is gone; now on net P2_P: U5.E7 (P0_D11/TX_D5_P)
- net TX_D0_P is gone; now on net P2_N: U5.F8 (P0_D10/TX_D5_N)
- net TX_D1_N is gone; now on net Q4_P: U5.D7 (P0_D9/TX_D4_P)
- net TX_D1_P is gone; now on net Q4_N: U5.E8 (P0_D8/TX_D4_N)
- net TX_D2_N is gone; now on net P1_P: U5.D8 (P0_D7/TX_D3_P)
- net TX_D2_P is gone; now on net P1_N: U5.E9 (P0_D6/TX_D3_N)
- net TX_D3_N is gone; now on net Q2_P: U5.D9 (P0_D5/TX_D2_P)
- net TX_D3_P is gone; now on net Q2_N: U5.E10 (P0_D4/TX_D2_N)
- net TX_D4_N is gone; now on net P3_P: U5.D10 (P0_D3/TX_D1_P)
- net TX_D4_P is gone; now on net P3_N: U5.E11 (P0_D2/TX_D1_N)
- net TX_D5_N is gone; now on net P4_P: U5.D11 (P0_D1/TX_D0_P)
- net TX_D5_P is gone; now on net P4_N: U5.E12 (P0_D0/TX_D0_N)
- net TX_FRAME_N is gone; now on net Q1_N: U5.H9 (TX_FRAME_N)
- net TX_FRAME_P is gone; now on net Q1_P: U5.G9 (TX_FRAME_P)
- net DATA_CLK_N: now also R9.2, U4.3 (B); no longer HDMI2.9 (DATA0-)
- net DATA_CLK_P: now also R9.1, U4.2 (A); no longer HDMI2.7 (DATA0+)
- net GND: now also C10.2, C11.2, C4.2, C5.2, C6.2, C7.2, C8.2, C9.2, U10.5 (GND), U13.5 (GND), U3.5 (GND), U4.5 (GND), U6.5 (GND), U7.5 (GND), U8.5 (GND), U9.5 (GND)
- net RX_D0_N: now also R13.2, U9.3 (B); no longer HDMI1.9 (DATA0-)
- net RX_D0_P: now also R13.1, U9.2 (A); no longer HDMI1.7 (DATA0+)
- net RX_D1_N: now also R8.2, U3.3 (B); no longer HDMI2.6 (DATA1-)
- net RX_D1_P: now also R8.1, U3.2 (A); no longer HDMI2.4 (DATA1+)
- net RX_D2_N: now also R15.2, U13.3 (B); no longer HDMI1.3 (DATA2-)
- net RX_D2_P: now also R15.1, U13.2 (A); no longer HDMI1.1 (DATA2+)
- net RX_D3_N: now also R10.2, U6.3 (B); no longer HDMI2.12 (CLK-)
- net RX_D3_P: now also R10.1, U6.2 (A); no longer HDMI2.10 (CLK+)
- net RX_D4_N: now also R12.2, U8.3 (B); no longer HDMI1.6 (DATA1-)
- net RX_D4_P: now also R12.1, U8.2 (A); no longer HDMI1.4 (DATA1+)
- net RX_D5_N: now also R14.2, U10.3 (B); no longer HDMI1.12 (CLK-)
- net RX_D5_P: now also R14.1, U10.2 (A); no longer HDMI1.10 (CLK+)
- net RX_FRAME_N: now also R11.2, U7.3 (B); no longer HDMI2.3 (DATA2-)
- net RX_FRAME_P: now also R11.1, U7.2 (A); no longer HDMI2.1 (DATA2+)
- net VCC_3V3: now also C10.1, C11.1, C4.1, C5.1, C6.1, C7.1, C8.1, C9.1, U10.8 (Vcc), U13.8 (Vcc), U3.8 (Vcc), U4.8 (Vcc), U6.8 (Vcc), U7.8 (Vcc), U8.8 (Vcc), U9.8 (Vcc)
- net XTAL1V8: now also R16.2
- net XTAL1V8_IN: now reaches C152.2, X4.3 (OUT)
- net XTAL1V8_IN: now also R16.1
- removed net IO10: J2J3.10
- removed net IO11: J2J3.11
- removed net IO12: J2J3.12
- removed net IO13: J2J3.13
- removed net IO14: J2J3.14
- removed net IO15: J2J3.15
- removed net IO16: J2J3.16
- removed net IO9: J2J3.9
- new net TMDS_CLK_N: HDMI1.12 (CLK-), U4.6 (Z)
- new net TMDS_CLK_P: HDMI1.10 (CLK+), U4.7 (Y)
- new net TMDS_D0_N: HDMI2.6 (DATA1-), U9.6 (Z)
- new net TMDS_D0_P: HDMI2.4 (DATA1+), U9.7 (Y)
- new net TMDS_D1_N: HDMI1.6 (DATA1-), U3.6 (Z)
- new net TMDS_D1_P: HDMI1.4 (DATA1+), U3.7 (Y)
- new net TMDS_D2_N: HDMI2.12 (CLK-), U13.6 (Z)
- new net TMDS_D2_P: HDMI2.10 (CLK+), U13.7 (Y)
- new net TMDS_D3_N: HDMI1.3 (DATA2-), U6.6 (Z)
- new net TMDS_D3_P: HDMI1.1 (DATA2+), U6.7 (Y)
- new net TMDS_D4_N: HDMI2.9 (DATA0-), U8.6 (Z)
- new net TMDS_D4_P: HDMI2.7 (DATA0+), U8.7 (Y)
- new net TMDS_D5_N: HDMI2.3 (DATA2-), U10.6 (Z)
- new net TMDS_D5_P: HDMI2.1 (DATA2+), U10.7 (Y)
- new net TMDS_FRAME_N: HDMI1.9 (DATA0-), U7.6 (Z)
- new net TMDS_FRAME_P: HDMI1.7 (DATA0+), U7.7 (Y)
- no-connect marks 22 -> 38
Other:
- note added: "LVDS RX"
- note added: "LVDS TX"
- note removed: "1.5V unused"
- note removed: "Short C and leave pullups open"
- moved on the sheet: 1V8G1, 3V3G1, 5V0G1, 7020to9363_8, 9363to7020_8, C1, C14, C142, C143, C144, C145, C146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

Commit message: V1.2 update
Parts:
- removed C11, C9: 0.1μ, PYNQSDR:LC-0402_C, symbol pynqsdr-altium-import:1_CAP_2
- removed C14, C168, C176: 1μ, PYNQSDR:LC-0402_C, symbol pynqsdr-altium-import:3_CAP_1
- removed C15, C169, C171, C173: 0.001μ, PYNQSDR:LC-0402_C, symbol pynqsdr-altium-import:3_CAP_1
- removed C162, C165: 10μ, PYNQSDR:LC-0402_C, symbol pynqsdr-altium-import:3_CAP_1
- removed RX1, RX3: JCCEM001, PYNQSDR:CNSMARAL687W375H171, symbol pynqsdr-altium-import:2_JCCEM001
- removed TX1: JCCEM001, PYNQSDR:CNSMARAL687W375H171, symbol pynqsdr-altium-import:0_JCCEM001
- added C2: 0.1μ, PYNQSDR:LC-0402_C, symbol pynqsdr-altium-import:3_CAP_2
- added C3: NC, PYNQSDR:LC-0402_C, symbol pynqsdr-altium-import:3_CAP_2
- added R1: NC, PYNQSDR:LC-0402_R, symbol pynqsdr-altium-import:2_RES_1
- added RX1, RX3, TX1: Conn_Coaxial, Connector_Coaxial:SMA_Amphenol_132289_EdgeMount, symbol Connector:Conn_Coaxial
- added X2: TCXO, Crystal:Crystal_SMD_7050-4Pin_7.0x5.0mm, symbol pynqsdr-altium-import:0_XTAL-4
- U10, U13, U3, U4, U6, U7, U8, U9: footprint Package_SO:TSSOP-8_4.4x3mm_P0.65mm -> Package_SO:TSSOP-8_3x3mm_P0.65mm
Connections:
- net GND: now also C2.1, C3.1, X2.2 (GND)
- net OI2: now also R1.1
- net RFGND2: now also RX3.2 (Ext)
- net RFGND3: now also RX1.2 (Ext)
- net RFGND4: now also TX1.2 (Ext)
- net VCC_3V3: now also C2.2, C3.2, X2.4 (VCC)
- net at RX_SMT2.3 (SIG): now also RX1.1 (In)
- net at TX_SMT2.3 (SIG): now also TX1.1 (In)
- net at RX_SMT1.3 (SIG): now also RX3.1 (In)
- new net: R1.2, X2.3 (OUT)
Other:
- note added: "Fly a wire to use 1.8 V Xtal / 5032 Xtal"
- note added: "Fly a wire to use 1.8 V Xtal / bigger Xtal"
- note removed: "Fly a wire to use 3.3 V Xtal"
- moved on the sheet: RX_SMT2
